File: VolcaModularMidi.kicad_sch (KiCad schematic)
At the start: 6 parts, among them J1 Conn_01x04_Male, J2 MIDI_IN, U1 6N137

Commit message: Finished routing and laying out pcb
Parts:
- removed J1: Conn_01x04_Male, Connector_PinHeader_2.54mm:PinHeader_1x04_P2.54mm_Vertical, symbol Connector:Conn_01x04_Male
- added J1: Conn_01x03_Female, Connector_PinSocket_2.00mm:PinSocket_1x03_P2.00mm_Vertical, symbol Connector:Conn_01x03_Female
- J2: footprint SensaiLib:din-5 -> eurocad:MIDI_DIN5
- U1: footprint Package_DIP:DIP-8_W7.62mm -> Package_DIP:DIP-8_W7.62mm_LongPads
Connections:
- net GND: now also J1.3 (Pin_3)
- net RX: now also J1.2 (Pin_2)
- net +3V3 renamed VCC
- net VCC: now also J1.1 (Pin_1)

Commit message: Added mounting holes, replaced jumper connector with jst connector
Parts:
- J1: footprint Connector_PinSocket_2.00mm:PinSocket_1x03_P2.00mm_Vertical -> Connector_JST:JST_EH_B3B-EH-A_1x03_P2.50mm_Vertical
Changed lines of the file:
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@@
       (effects (font (size 1.27 1.27)) (justify left))
     )
-    (property "Footprint" "Connector_PinSocket_2.00mm:PinSocket_1x03_P2.00mm_Vertical" (id 2) (at 50.8 27.94 0)
+    (property "Footprint" "Connector_JST:JST_EH_B3B-EH-A_1x03_P2.50mm_Vertical" (id 2) (at 50.8 27.94 0)
       (effects (font (size 1.27 1.27)) hide)
     )
@@
     )
     (path "/54642827-47cd-4706-b98a-56254729af31"
-      (reference "J1") (unit 1) (value "Conn_01x03_Female") (footprint "Connector_PinSocket_2.00mm:PinSocket_1x03_P2.00mm_Vertical")
+      (reference "J1") (unit 1) (value "Conn_01x03_Female") (footprint "Connector_JST:JST_EH_B3B-EH-A_1x03_P2.50mm_Vertical")
     )
     (path "/00000000-0000-0000-0000-00005cd053d1"
